File: kicad/kingslayer-28/kingslayer-28.kicad_sch (KiCad schematic)
At the start: 67 parts, among them IC1 STM32F303CCT7, K1 KEYSW, K10 KEYSW, K11 KEYSW, K12 KEYSW, K13 KEYSW, K14 KEYSW, K15 KEYSW, K16 KEYSW, K17 KEYSW, K18 KEYSW, K19 KEYSW, K2 KEYSW, K20 KEYSW, K21 KEYSW, K22 KEYSW, K23 KEYSW, K24 KEYSW, K25 KEYSW, K26 KEYSW, K27 KEYSW, K28 KEYSW, K3 KEYSW, K4 KEYSW, K5 KEYSW, K6 KEYSW, K7 KEYSW, K8 KEYSW, K9 KEYSW, Y1 FA-238_16.0000MB-C3

Commit message: MCU done...
Parts:
- removed Y1: FA-238_16.0000MB-C3, FA238160000MBC3, symbol FA-238_16.0000MB-C3:FA-238_16.0000MB-C3
- added C10: 100n, symbol Device:C_Small
- added R1: 10k, symbol keyboard_parts:R
- added SW1: SW_SPDT, symbol Switch:SW_SPDT
- added X1: 8Mhz, symbol keyboard_parts:XTAL_GND
- C3, C4, C5, C6: value 0.1u -> 100n
Connections:
- net VCC is gone; now on net +5V: IC1.1 (VBAT), IC1.24 (VDD_1), IC1.36 (VDD_2), IC1.48 (VDD_3), IC1.9 (VDDA)
- net +5V: now also C10.1, SW1.1 (A), SW1.3 (C), X1.3
- net boot0: now also R1.2
- net col0: now also IC1.15 (PA5); no longer IC1.29 (PA8)
- net col1: now also IC1.16 (PA6); no longer IC1.28 (PB15)
- net col2: now also IC1.17 (PA7); no longer IC1.27 (PB14)
- net col3: now also IC1.18 (PB0); no longer IC1.26 (PB13)
- net col4: now also IC1.19 (PB1); no longer IC1.25 (PB12)
- net col5: now also IC1.20 (PB2); no longer IC1.38 (PA15)
- net col6: now also IC1.21 (PB10); no longer IC1.37 (PA14)
- net nrst: now also S1.2, S1.4, C10.2
- net row0: now also IC1.10 (PA0); no longer IC1.34 (PA13)
- net row1: now also IC1.11 (PA1); no longer IC1.33 (PA12)
- net row2: now also IC1.12 (PA2); no longer IC1.32 (PA11)
- net row3: now also IC1.13 (PA3); no longer IC1.31 (PA10)
- net row4: now also IC1.14 (PA4); no longer IC1.30 (PA9)
- net scl: now also IC1.38 (PA15); no longer IC1.40 (PB4)
- net sda: now also IC1.37 (PA14); no longer IC1.39 (PB3)
- net xtal1: now also X1.1
- net xtal2: now also X1.2
- new net: R1.1, SW1.2 (B)
- new net dm: IC1.32 (PA11)
- new net dp: IC1.33 (PA12)
- no-connect marks 3 -> 19
Other:
- note removed: "?"
- note removed: "This will need to be 8MHZ I think"
- moved on the sheet: C1, C2, C3, C4, C5, C6, C7, S1

Commit message: done I guess
Parts:
- added C11: 0.47u, symbol Device:C_Small
- added C12: 33u, symbol Device:C_Small
- added IC3: LM3940IMP-3.3_NOPB, SOT230P700X180-4N, symbol LM3940IMP-3.3_NOPB:LM3940IMP-3.3_NOPB
- added R7, R8: 5.1k, symbol keyboard_parts:R
- C1, C2: value 22p -> 20p
- SW1: value SW_SPDT -> MSS13PLP
- X1: value 8Mhz -> IC21008.000M30.0EE1B
Connections:
- net +5V: now also USB1.A1 (GND), USB1.A12 (GND), USB1.A4 (VBUS), USB1.A9 (VBUS), USB1.B1 (GND), USB1.B12 (GND), USB1.B4 (VBUS), USB1.B9 (VBUS), USB1.S1 (Shell1), USB1.S2 (Shell2), USB1.S3 (Shell3), USB1.S4 (Shell4), C11.1, C11.2, C12.1, C12.2, IC3.1 (IN), IC3.2 (GND_1), IC3.3 (OUT), IC3.4 (GND_2), R7.2, R8.2
- net dm: now also USB1.A6 (D+), USB1.B6 (D+)
- net dp: now also USB1.A7 (D-), USB1.B7 (D-)
- net at USB1.A5 (CC1): now also R7.1
- net at USB1.B5 (CC2): now also R8.1
- no-connect marks 19 -> 30
Other:
- moved on the sheet: USB1

Commit message: add info
Other:
- note added: "Diodes are 1N4148W RHG"
Changed lines of the file:
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@@
     (effects (font (size 1.27 1.27)) (justify left top))
+  )
+  (text "Diodes are 1N4148W RHG" (at 148.59 86.36 0)
+    (effects (font (size 1.27 1.27)) (justify left bottom))
   )
   (global_label "col3" (shape input) (at 100.33 20.32 90) (fields_autoplaced)

Commit message: oops
Connections:
- net dm: now also USB1.A7 (D-), USB1.B7 (D-); no longer USB1.A6 (D+), USB1.B6 (D+)
- net dp: now also USB1.A6 (D+), USB1.B6 (D+); no longer USB1.A7 (D-), USB1.B7 (D-)
- no-connect marks 30 -> 29
Changed lines of the file:
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@@
   (no_connect (at 60.96 134.62))
   (no_connect (at 190.5 104.14))
-  (no_connect (at 207.01 121.92))
   (no_connect (at 60.96 137.16))
   (no_connect (at 87.63 109.22))
@@
     (stroke (width 0) (type default))
   )
-  (wire (pts (xy 281.94 113.03) (xy 281.94 123.19))
-    (stroke (width 0) (type default))
-  )
   (wire (pts (xy 229.87 33.02) (xy 237.49 33.02))
     (stroke (width 0) (type default))
@@
     (stroke (width 0) (type default))
   )
-  (wire (pts (xy 281.94 113.03) (xy 283.21 113.03))
-    (stroke (width 0) (type default))
-  )
   (wire (pts (xy 43.18 71.12) (xy 43.18 72.39))
     (stroke (width 0) (type default))
@@
     (stroke (width 0) (type default))
   )
+  (wire (pts (xy 283.21 123.19) (xy 283.21 113.03))
+    (stroke (width 0) (type default))
+  )
   (wire (pts (xy 100.33 109.22) (xy 100.33 111.76))
     (stroke (width 0) (type default))
@@
     (stroke (width 0) (type default))
   )
-  (wire (pts (xy 281.94 123.19) (xy 241.3 123.19))
+  (wire (pts (xy 241.3 123.19) (xy 283.21 123.19))
     (stroke (width 0) (type default))
   )
@@
     )
   )
-  (global_label "dp" (shape input) (at 190.5 140.97 180) (fields_autoplaced)
-    (effects (font (size 1.27 1.27)) (justify right))
-    (property "Intersheetrefs" "${INTERSHEET_REFS}" (at 185.2168 140.97 0)
-      (effects (font (size 1.27 1.27)) (justify right) hide)
-    )
-  )
   (global_label "col5" (shape input) (at 90.17 177.8 270) (fields_autoplaced)
     (effects (font (size 1.27 1.27)) (justify right))
@@
     )
   )
+  (global_label "dp" (shape input) (at 190.5 135.89 180) (fields_autoplaced)
+    (effects (font (size 1.27 1.27)) (justify right))
+    (property "Intersheetrefs" "${INTERSHEET_REFS}" (at 185.2168 135.89 0)
+      (effects (font (size 1.27 1.27)) (justify right) hide)
+    )
+  )
   (global_label "xtal1" (shape input) (at 62.23 139.7 180) (fields_autoplaced)
     (effects (font (size 1.27 1.27)) (justify right))
@@
     )
   )
-  (global_label "dm" (shape input) (at 190.5 135.89 180) (fields_autoplaced)
-    (effects (font (size 1.27 1.27)) (justify right))
-    (property "Intersheetrefs" "${INTERSHEET_REFS}" (at 184.6725 135.89 0)
-      (effects (font (size 1.27 1.27)) (justify right) hide)
-    )
-  )
   (global_label "row4" (shape input) (at 20.32 85.09 180) (fields_autoplaced)
     (effects (font (size 1.27 1.27)) (justify right))
@@
     )
   )
+  (global_label "dm" (shape input) (at 190.5 140.97 180) (fields_autoplaced)
+    (effects (font (size 1.27 1.27)) (justify right))
+    (property "Intersheetrefs" "${INTERSHEET_REFS}" (at 184.6725 140.97 0)
+      (effects (font (size 1.27 1.27)) (justify right) hide)
+    )
+  )

Commit message: Addressed some comments
Connections:
- net scl: now also IC1.45 (PB8); no longer IC1.38 (PA15)
- net sda: now also IC1.46 (PB9); no longer IC1.37 (PA14)
Other:
- note added: "PA13 = SWDIO PA14 = SWCLK might want to expose those"
- moved on the sheet: C1, C10, C11, C12, C2, C3, C4, C5, C6, C7, IC1, IC3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

Commit message: update pics
Parts:
- D1, D10, D11, D12, D13, D14, D15, D16, D17, D18, D19, D2, D20, D21, D22, D23, D24, D25, D26, D27, D28, D3, D4, D5, D6, D7, D8, D9: value D -> 1N4148W RHG
Connections:
- net scl renamed RGB/scl
- net sda renamed RGB/sda
Other:
- sheet RGB ports: added scl, sda; removed none
- note removed: "Diodes are 1N4148W RHG"

Commit message: Update after watching phil
Parts:
- added J1: Conn_01x04_Pin, symbol Connector:Conn_01x04_Pin
- added R9: 1k5, symbol keyboard_parts:R
Connections:
- net +5V: now also J1.1 (Pin_1), J1.4 (Pin_4), R9.1; no longer USB1.S1 (Shell1), USB1.S2 (Shell2), USB1.S3 (Shell3), USB1.S4 (Shell4)
- net swdio: now reaches IC1.34 (PA13)
- net swdio: now also J1.3 (Pin_3)
- net swclk: now reaches IC1.37 (PA14)
- net swclk: now also J1.2 (Pin_2)
- net dm renamed d-
- net dp renamed d+
- net d+: now also R9.2
- no-connect marks 29 -> 31
Other:
- note added: "8MHz Crystal"
- note added: "Button that resets the MCU"
- note added: "Switch that flips BOOT0"
- note added: "Voltage regulator that converts 5v to 3v3"
- note removed: "PA13 = SWDIO PA14 = SWCLK might want to expose those"
- moved on the sheet: SW1

Commit message: ground shield
Connections:
- net +5V: now also USB1.S1 (Shell1), USB1.S2 (Shell2), USB1.S3 (Shell3), USB1.S4 (Shell4)
- no-connect marks 31 -> 27
Changed lines of the file:
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@@
   (junction (at 120.65 64.77) (diameter 0) (color 0 0 0 0)
   )
+  (junction (at 218.44 67.31) (diameter 0) (color 0 0 0 0)
+  )
   (junction (at 76.2 106.68) (diameter 0) (color 0 0 0 0)
   )
@@
   (junction (at 220.98 40.64) (diameter 0) (color 0 0 0 0)
   )
+  (junction (at 218.44 64.77) (diameter 0) (color 0 0 0 0)
+  )
   (junction (at 59.69 52.07) (diameter 0) (color 0 0 0 0)
   )
@@
   (junction (at 189.23 63.5) (diameter 0) (color 0 0 0 0)
   )
+  (junction (at 218.44 62.23) (diameter 0) (color 0 0 0 0)
+  )
   (junction (at 140.97 26.67) (diameter 0) (color 0 0 0 0)
+  )
+  (junction (at 218.44 69.85) (diameter 0) (color 0 0 0 0)
   )
   (junction (at 165.1 139.7) (diameter 0) (color 0 0 0 0)
@@
   (no_connect (at 154.94 154.94))
   (no_connect (at 186.69 39.37))
-  (no_connect (at 218.44 64.77))
   (no_connect (at 137.16 111.76))
   (no_connect (at 129.54 111.76))
-  (no_connect (at 218.44 62.23))
   (no_connect (at 154.94 157.48))
   (no_connect (at 186.69 36.83))
@@
   (no_connect (at 105.41 139.7))
   (no_connect (at 132.08 111.76))
-  (no_connect (at 218.44 69.85))
   (no_connect (at 154.94 147.32))
   (no_connect (at 186.69 49.53))
@@
   (no_connect (at 139.7 111.76))
   (no_connect (at 154.94 149.86))
-  (no_connect (at 218.44 67.31))
   (no_connect (at 139.7 180.34))
   (no_connect (at 154.94 160.02))
@@
     (stroke (width 0) (type default))
   )
+  (wire (pts (xy 218.44 62.23) (xy 218.44 57.15))
+    (stroke (width 0) (type default))
+  )
   (wire (pts (xy 120.65 77.47) (xy 119.38 77.47))
     (stroke (width 0) (type default))
@@
     (stroke (width 0) (type default))
   )
+  (wire (pts (xy 218.44 69.85) (xy 218.44 67.31))
+    (stroke (width 0) (type default))
+  )
   (wire (pts (xy 119.38 26.67) (xy 120.65 26.67))
     (stroke (width 0) (type default))
@@
     (stroke (width 0) (type default))
   )
+  (wire (pts (xy 218.44 64.77) (xy 218.44 62.23))
+    (stroke (width 0) (type default))
+  )
   (wire (pts (xy 134.62 180.34) (xy 134.62 177.8))
     (stroke (width 0) (type default))
@@
     (stroke (width 0) (type default))
   )
+  (wire (pts (xy 218.44 67.31) (xy 218.44 64.77))
+    (stroke (width 0) (type default))
+  )
   (wire (pts (xy 120.65 64.77) (xy 119.38 64.77))
     (stroke (width 0) (type default))
@@
   )
   (wire (pts (xy 33.02 102.87) (xy 39.37 102.87))
+    (stroke (width 0) (type default))
+  )
+  (wire (pts (xy 218.44 72.39) (xy 218.44 69.85))
     (stroke (width 0) (type default))
   )
@@
     )
   )
-  (symbol (lib_id "keyboard_parts:GND") (at 218.44 57.15 0) (unit 1)
+  (symbol (lib_id "keyboard_parts:GND") (at 218.44 72.39 0) (unit 1)
     (in_bom yes) (on_board yes) (dnp no)
-    (property "Reference" "#PWR023" (at 218.44 55.88 0)
+    (property "Reference" "#PWR023" (at 218.44 71.12 0)
       (effects (font (size 0.508 0.508)) hide)
     )
-    (property "Value" "GND" (at 218.44 59.69 0)
+    (property "Value" "GND" (at 218.44 74.93 0)
       (effects (font (size 0.762 0.762)))
     )
-    (property "Footprint" "" (at 218.44 57.15 0)
-      (effects (font (size 1.524 1.524)))
-    )
-    (property "Datasheet" "" (at 218.44 57.15 0)
-      (effects (font (size 1.524 1.524)))
-    )
+    (property "Footprint" "" (at 218.44 72.39 0)
+      (effects (font (size 1.524 1.524)))
+    )
+    (property "Datasheet" "" (at 218.44 72.39 0)
+      (effects (font (size 1.524 1.524)))
+    )
