File: kicad/kingslayer-28/rgb.kicad_sch (KiCad schematic)
At the start: 36 parts, among them IC2 IS31FL3731-QFLS2-TR

Commit message: initial placement
Connections:
- net +5V: no longer C8.2, C9.2, IC2.18 (AD), IC2.29 (PAD), IC2.5 (GND), R2.2, R3.1, R4.1, R5.1, R6.2
- new net +3V3: R3.1, R4.1, R5.1
- new net GND: C8.2, C9.2, IC2.18 (AD), IC2.29 (PAD), IC2.5 (GND), R2.2, R6.2
Changed lines of the file:
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@@
     )
   )
-  (symbol (lib_id "keyboard_parts:+3V3") (at 190.5 119.38 0) (unit 1)
+  (symbol (lib_id "power:+3V3") (at 190.5 119.38 0) (unit 1)
     (in_bom yes) (on_board yes) (dnp no) (fields_autoplaced)
     (property "Reference" "#PWR018" (at 190.5 120.142 0)
@@
     )
     (property "Footprint" "" (at 190.5 119.38 0)
-      (effects (font (size 1.524 1.524)))
+      (effects (font (size 1.27 1.27)) hide)
     )
     (property "Datasheet" "" (at 190.5 119.38 0)
-      (effects (font (size 1.524 1.524)))
+      (effects (font (size 1.27 1.27)) hide)
     )
     (pin "1")
@@
     )
   )
-  (symbol (lib_id "keyboard_parts:+5V") (at 193.04 55.88 0) (unit 1)
+  (symbol (lib_id "power:+5V") (at 193.04 55.88 0) (unit 1)
     (in_bom yes) (on_board yes) (dnp no)
     (property "Reference" "#PWR017" (at 193.04 56.642 0)
@@
     )
     (property "Footprint" "" (at 193.04 55.88 0)
-      (effects (font (size 1.524 1.524)))
+      (effects (font (size 1.27 1.27)) hide)
     )
     (property "Datasheet" "" (at 193.04 55.88 0)
-      (effects (font (size 1.524 1.524)))
+      (effects (font (size 1.27 1.27)) hide)
     )
     (pin "1")
@@
     )
   )
-  (symbol (lib_id "keyboard_parts:GND") (at 190.5 152.4 0) (unit 1)
+  (symbol (lib_id "power:GND") (at 190.5 152.4 0) (unit 1)
     (in_bom yes) (on_board yes) (dnp no)
     (property "Reference" "#PWR019" (at 190.5 151.13 0)
@@
     )
     (property "Footprint" "" (at 190.5 152.4 0)
-      (effects (font (size 1.524 1.524)))
+      (effects (font (size 1.27 1.27)) hide)
     )
     (property "Datasheet" "" (at 190.5 152.4 0)
-      (effects (font (size 1.524 1.524)))
+      (effects (font (size 1.27 1.27)) hide)
     )
     (pin "1")
@@
     )
   )
-  (symbol (lib_id "keyboard_parts:GND") (at 254 139.7 0) (unit 1)
+  (symbol (lib_id "power:GND") (at 254 139.7 0) (unit 1)
     (in_bom yes) (on_board yes) (dnp no)
     (property "Reference" "#PWR015" (at 254 138.43 0)
@@
     )
     (property "Footprint" "" (at 254 139.7 0)
-      (effects (font (size 1.524 1.524)))
+      (effects (font (size 1.27 1.27)) hide)
     )
     (property "Datasheet" "" (at 254 139.7 0)
-      (effects (font (size 1.524 1.524)))
+      (effects (font (size 1.27 1.27)) hide)
     )
     (pin "1")
@@
     )
   )
-  (symbol (lib_id "keyboard_parts:GND") (at 215.9 35.56 0) (unit 1)
+  (symbol (lib_id "power:GND") (at 215.9 35.56 0) (unit 1)
     (in_bom yes) (on_board yes) (dnp no)
     (property "Reference" "#PWR020" (at 215.9 34.29 0)
@@
     )
     (property "Footprint" "" (at 215.9 35.56 0)
-      (effects (font (size 1.524 1.524)))
+      (effects (font (size 1.27 1.27)) hide)
     )
     (property "Datasheet" "" (at 215.9 35.56 0)
-      (effects (font (size 1.524 1.524)))
+      (effects (font (size 1.27 1.27)) hide)
     )
     (pin "1")
@@
     )
   )
-  (symbol (lib_id "keyboard_parts:GND") (at 201.93 63.5 0) (unit 1)
+  (symbol (lib_id "power:GND") (at 201.93 63.5 0) (unit 1)
     (in_bom yes) (on_board yes) (dnp no)
     (property "Reference" "#PWR021" (at 201.93 62.23 0)
@@
     )
     (property "Footprint" "" (at 201.93 63.5 0)
-      (effects (font (size 1.524 1.524)))
+      (effects (font (size 1.27 1.27)) hide)
     )
     (property "Datasheet" "" (at 201.93 63.5 0)
-      (effects (font (size 1.524 1.524)))
+      (effects (font (size 1.27 1.27)) hide)
     )
     (pin "1")
@@
     )
   )
-  (symbol (lib_id "keyboard_parts:GND") (at 252.73 60.96 0) (unit 1)
+  (symbol (lib_id "power:GND") (at 252.73 60.96 0) (unit 1)
     (in_bom yes) (on_board yes) (dnp no)
     (property "Reference" "#PWR030" (at 252.73 59.69 0)
@@
     )
     (property "Footprint" "" (at 252.73 60.96 0)
-      (effects (font (size 1.524 1.524)))
+      (effects (font (size 1.27 1.27)) hide)
     )
     (property "Datasheet" "" (at 252.73 60.96 0)
-      (effects (font (size 1.524 1.524)))
+      (effects (font (size 1.27 1.27)) hide)
     )
     (pin "1")
@@
     )
   )
-  (symbol (lib_id "keyboard_parts:GND") (at 193.04 45.72 0) (unit 1)
+  (symbol (lib_id "power:GND") (at 193.04 45.72 0) (unit 1)
     (in_bom yes) (on_board yes) (dnp no)
     (property "Reference" "#PWR016" (at 193.04 44.45 0)
@@
     )
     (property "Footprint" "" (at 193.04 45.72 0)
-      (effects (font (size 1.524 1.524)))
+      (effects (font (size 1.27 1.27)) hide)
     )
     (property "Datasheet" "" (at 193.04 45.72 0)
-      (effects (font (size 1.524 1.524)))
-    )
-    (pin "1")
+      (effects (font (size 1.27 1.27)) hide)
+    )
+    (pin "1")

Commit message: revert footprints, finalize placement
Parts:
- D29, D30, D31, D32, D33, D34, D35, D36, D37, D38, D39, D40, D41, D42, D43, D44, D45, D46, D47, D48, D49, D50, D51, D52, D53, D54, D55, D56: footprint LED_SMD:LED_RGB_1210 -> acheron_Components:LED_RGB_SMD_6028_2.8x3.5mm
Changed lines of the file:
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@@
       (effects (font (size 1.27 1.27)) (justify left))
     )
-    (property "Footprint" "LED_SMD:LED_RGB_1210" (at 76.2 78.74 0)
+    (property "Footprint" "acheron_Components:LED_RGB_SMD_6028_2.8x3.5mm" (at 76.2 78.74 0)
       (effects (font (size 1.27 1.27)) hide)
     )
@@
       (effects (font (size 1.27 1.27)) (justify left))
     )
-    (property "Footprint" "LED_SMD:LED_RGB_1210" (at 57.15 111.76 0)
+    (property "Footprint" "acheron_Components:LED_RGB_SMD_6028_2.8x3.5mm" (at 57.15 111.76 0)
       (effects (font (size 1.27 1.27)) hide)
     )
@@
       (effects (font (size 1.27 1.27)) (justify left))
     )
-    (property "Footprint" "LED_SMD:LED_RGB_1210" (at 95.25 111.76 0)
+    (property "Footprint" "acheron_Components:LED_RGB_SMD_6028_2.8x3.5mm" (at 95.25 111.76 0)
       (effects (font (size 1.27 1.27)) hide)
     )
@@
       (effects (font (size 1.27 1.27)) (justify left))
     )
-    (property "Footprint" "LED_SMD:LED_RGB_1210" (at 57.15 78.74 0)
+    (property "Footprint" "acheron_Components:LED_RGB_SMD_6028_2.8x3.5mm" (at 57.15 78.74 0)
       (effects (font (size 1.27 1.27)) hide)
     )
@@
       (effects (font (size 1.27 1.27)) (justify left))
     )
-    (property "Footprint" "LED_SMD:LED_RGB_1210" (at 38.1 144.78 0)
+    (property "Footprint" "acheron_Components:LED_RGB_SMD_6028_2.8x3.5mm" (at 38.1 144.78 0)
       (effects (font (size 1.27 1.27)) hide)
     )
@@
       (effects (font (size 1.27 1.27)) (justify left))
     )
-    (property "Footprint" "LED_SMD:LED_RGB_1210" (at 57.15 45.72 0)
+    (property "Footprint" "acheron_Components:LED_RGB_SMD_6028_2.8x3.5mm" (at 57.15 45.72 0)
       (effects (font (size 1.27 1.27)) hide)
     )
@@
       (effects (font (size 1.27 1.27)) (justify left))
     )
-    (property "Footprint" "LED_SMD:LED_RGB_1210" (at 38.1 45.72 0)
+    (property "Footprint" "acheron_Components:LED_RGB_SMD_6028_2.8x3.5mm" (at 38.1 45.72 0)
       (effects (font (size 1.27 1.27)) hide)
     )
@@
       (effects (font (size 1.27 1.27)) (justify left))
     )
-    (property "Footprint" "LED_SMD:LED_RGB_1210" (at 99.06 177.8 0)
+    (property "Footprint" "acheron_Components:LED_RGB_SMD_6028_2.8x3.5mm" (at 99.06 177.8 0)
       (effects (font (size 1.27 1.27)) hide)
     )
@@
       (effects (font (size 1.27 1.27)) (justify left))
     )
-    (property "Footprint" "LED_SMD:LED_RGB_1210" (at 133.35 144.78 0)
+    (property "Footprint" "acheron_Components:LED_RGB_SMD_6028_2.8x3.5mm" (at 133.35 144.78 0)
       (effects (font (size 1.27 1.27)) hide)
     )
@@
       (effects (font (size 1.27 1.27)) (justify left))
     )
-    (property "Footprint" "LED_SMD:LED_RGB_1210" (at 57.15 177.8 0)
+    (property "Footprint" "acheron_Components:LED_RGB_SMD_6028_2.8x3.5mm" (at 57.15 177.8 0)
       (effects (font (size 1.27 1.27)) hide)
     )
@@
       (effects (font (size 1.27 1.27)) (justify left))
     )
-    (property "Footprint" "LED_SMD:LED_RGB_1210" (at 118.11 177.8 0)
+    (property "Footprint" "acheron_Components:LED_RGB_SMD_6028_2.8x3.5mm" (at 118.11 177.8 0)
       (effects (font (size 1.27 1.27)) hide)
     )
@@
       (effects (font (size 1.27 1.27)) (justify left))
     )
-    (property "Footprint" "LED_SMD:LED_RGB_1210" (at 38.1 111.76 0)
+    (property "Footprint" "acheron_Components:LED_RGB_SMD_6028_2.8x3.5mm" (at 38.1 111.76 0)
       (effects (font (size 1.27 1.27)) hide)
     )
@@
       (effects (font (size 1.27 1.27)) (justify left))
     )
-    (property "Footprint" "LED_SMD:LED_RGB_1210" (at 114.3 111.76 0)
+    (property "Footprint" "acheron_Components:LED_RGB_SMD_6028_2.8x3.5mm" (at 114.3 111.76 0)
       (effects (font (size 1.27 1.27)) hide)
     )
@@
       (effects (font (size 1.27 1.27)) (justify left))
     )
-    (property "Footprint" "LED_SMD:LED_RGB_1210" (at 99.06 78.74 0)
+    (property "Footprint" "acheron_Components:LED_RGB_SMD_6028_2.8x3.5mm" (at 99.06 78.74 0)
       (effects (font (size 1.27 1.27)) hide)
     )
@@
       (effects (font (size 1.27 1.27)) (justify left))
     )
-    (property "Footprint" "LED_SMD:LED_RGB_1210" (at 114.3 45.72 0)
+    (property "Footprint" "acheron_Components:LED_RGB_SMD_6028_2.8x3.5mm" (at 114.3 45.72 0)
       (effects (font (size 1.27 1.27)) hide)
     )
@@
       (effects (font (size 1.27 1.27)) (justify left))
     )
-    (property "Footprint" "LED_SMD:LED_RGB_1210" (at 133.35 45.72 0)
+    (property "Footprint" "acheron_Components:LED_RGB_SMD_6028_2.8x3.5mm" (at 133.35 45.72 0)
       (effects (font (size 1.27 1.27)) hide)
     )
@@
       (effects (font (size 1.27 1.27)) (justify left))
     )
-    (property "Footprint" "LED_SMD:LED_RGB_1210" (at 76.2 111.76 0)
+    (property "Footprint" "acheron_Components:LED_RGB_SMD_6028_2.8x3.5mm" (at 76.2 111.76 0)
       (effects (font (size 1.27 1.27)) hide)
     )
@@
       (effects (font (size 1.27 1.27)) (justify left))
     )
-    (property "Footprint" "LED_SMD:LED_RGB_1210" (at 95.25 144.78 0)
+    (property "Footprint" "acheron_Components:LED_RGB_SMD_6028_2.8x3.5mm" (at 95.25 144.78 0)
       (effects (font (size 1.27 1.27)) hide)
     )
@@
       (effects (font (size 1.27 1.27)) (justify left))
     )
-    (property "Footprint" "LED_SMD:LED_RGB_1210" (at 95.25 45.72 0)
+    (property "Footprint" "acheron_Components:LED_RGB_SMD_6028_2.8x3.5mm" (at 95.25 45.72 0)
       (effects (font (size 1.27 1.27)) hide)
     )
@@
       (effects (font (size 1.27 1.27)) (justify left))
     )
-    (property "Footprint" "LED_SMD:LED_RGB_1210" (at 76.2 144.78 0)
+    (property "Footprint" "acheron_Components:LED_RGB_SMD_6028_2.8x3.5mm" (at 76.2 144.78 0)
       (effects (font (size 1.27 1.27)) hide)
     )
@@
       (effects (font (size 1.27 1.27)) (justify left))
     )
-    (property "Footprint" "LED_SMD:LED_RGB_1210" (at 38.1 177.8 0)
+    (property "Footprint" "acheron_Components:LED_RGB_SMD_6028_2.8x3.5mm" (at 38.1 177.8 0)
       (effects (font (size 1.27 1.27)) hide)
     )
@@
       (effects (font (size 1.27 1.27)) (justify left))
     )
-    (property "Footprint" "LED_SMD:LED_RGB_1210" (at 76.2 45.72 0)
+    (property "Footprint" "acheron_Components:LED_RGB_SMD_6028_2.8x3.5mm" (at 76.2 45.72 0)
       (effects (font (size 1.27 1.27)) hide)
     )
@@
       (effects (font (size 1.27 1.27)) (justify left))
     )
-    (property "Footprint" "LED_SMD:LED_RGB_1210" (at 158.75 45.72 0)
+    (property "Footprint" "acheron_Components:LED_RGB_SMD_6028_2.8x3.5mm" (at 158.75 45.72 0)
       (effects (font (size 1.27 1.27)) hide)
     )
@@
       (effects (font (size 1.27 1.27)) (justify left))
     )
-    (property "Footprint" "LED_SMD:LED_RGB_1210" (at 118.11 78.74 0)
+    (property "Footprint" "acheron_Components:LED_RGB_SMD_6028_2.8x3.5mm" (at 118.11 78.74 0)
       (effects (font (size 1.27 1.27)) hide)
     )
@@
       (effects (font (size 1.27 1.27)) (justify left))
     )
-    (property "Footprint" "LED_SMD:LED_RGB_1210" (at 57.15 144.78 0)
+    (property "Footprint" "acheron_Components:LED_RGB_SMD_6028_2.8x3.5mm" (at 57.15 144.78 0)
       (effects (font (size 1.27 1.27)) hide)
     )
@@
       (effects (font (size 1.27 1.27)) (justify left))
     )
-    (property "Footprint" "LED_SMD:LED_RGB_1210" (at 114.3 144.78 0)
+    (property "Footprint" "acheron_Components:LED_RGB_SMD_6028_2.8x3.5mm" (at 114.3 144.78 0)
       (effects (font (size 1.27 1.27)) hide)
     )
@@
       (effects (font (size 1.27 1.27)) (justify left))
     )
-    (property "Footprint" "LED_SMD:LED_RGB_1210" (at 38.1 78.74 0)
+    (property "Footprint" "acheron_Components:LED_RGB_SMD_6028_2.8x3.5mm" (at 38.1 78.74 0)
       (effects (font (size 1.27 1.27)) hide)
     )
@@
       (effects (font (size 1.27 1.27)) (justify left))
     )
-    (property "Footprint" "LED_SMD:LED_RGB_1210" (at 76.2 177.8 0)
-      (effects (font (size 1.27 1.27)) hide)
-    )
+    (property "Footprint" "acheron_Components:LED_RGB_SMD_6028_2.8x3.5mm" (at 76.2 177.8 0)
+      (effects (font (size 1.27 1.27)) hide)
+    )

Commit message: backup
Parts:
- D29, D30, D31, D32, D33, D34, D35, D36, D37, D38, D39, D40, D41, D42, D43, D44, D45, D46, D47, D48, D49, D50, D51, D52, D53, D54, D55, D56: footprint acheron_Components:LED_RGB_SMD_6028_2.8x3.5mm -> acheron_Components:LED_RGB_SMD_6028_2.8x3.5mm_Square
Changed lines of the file:
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@@
       (effects (font (size 1.27 1.27)) (justify left))
     )
-    (property "Footprint" "acheron_Components:LED_RGB_SMD_6028_2.8x3.5mm" (at 76.2 78.74 0)
+    (property "Footprint" "acheron_Components:LED_RGB_SMD_6028_2.8x3.5mm_Square" (at 76.2 78.74 0)
       (effects (font (size 1.27 1.27)) hide)
     )
@@
       (effects (font (size 1.27 1.27)) (justify left))
     )
-    (property "Footprint" "acheron_Components:LED_RGB_SMD_6028_2.8x3.5mm" (at 57.15 111.76 0)
+    (property "Footprint" "acheron_Components:LED_RGB_SMD_6028_2.8x3.5mm_Square" (at 57.15 111.76 0)
       (effects (font (size 1.27 1.27)) hide)
     )
@@
       (effects (font (size 1.27 1.27)) (justify left))
     )
-    (property "Footprint" "acheron_Components:LED_RGB_SMD_6028_2.8x3.5mm" (at 95.25 111.76 0)
+    (property "Footprint" "acheron_Components:LED_RGB_SMD_6028_2.8x3.5mm_Square" (at 95.25 111.76 0)
       (effects (font (size 1.27 1.27)) hide)
     )
@@
       (effects (font (size 1.27 1.27)) (justify left))
     )
-    (property "Footprint" "acheron_Components:LED_RGB_SMD_6028_2.8x3.5mm" (at 57.15 78.74 0)
+    (property "Footprint" "acheron_Components:LED_RGB_SMD_6028_2.8x3.5mm_Square" (at 57.15 78.74 0)
       (effects (font (size 1.27 1.27)) hide)
     )
@@
       (effects (font (size 1.27 1.27)) (justify left))
     )
-    (property "Footprint" "acheron_Components:LED_RGB_SMD_6028_2.8x3.5mm" (at 38.1 144.78 0)
+    (property "Footprint" "acheron_Components:LED_RGB_SMD_6028_2.8x3.5mm_Square" (at 38.1 144.78 0)
       (effects (font (size 1.27 1.27)) hide)
     )
@@
       (effects (font (size 1.27 1.27)) (justify left))
     )
-    (property "Footprint" "acheron_Components:LED_RGB_SMD_6028_2.8x3.5mm" (at 57.15 45.72 0)
+    (property "Footprint" "acheron_Components:LED_RGB_SMD_6028_2.8x3.5mm_Square" (at 57.15 45.72 0)
       (effects (font (size 1.27 1.27)) hide)
     )
@@
       (effects (font (size 1.27 1.27)) (justify left))
     )
-    (property "Footprint" "acheron_Components:LED_RGB_SMD_6028_2.8x3.5mm" (at 38.1 45.72 0)
+    (property "Footprint" "acheron_Components:LED_RGB_SMD_6028_2.8x3.5mm_Square" (at 38.1 45.72 0)
       (effects (font (size 1.27 1.27)) hide)
     )
@@
       (effects (font (size 1.27 1.27)) (justify left))
     )
-    (property "Footprint" "acheron_Components:LED_RGB_SMD_6028_2.8x3.5mm" (at 99.06 177.8 0)
+    (property "Footprint" "acheron_Components:LED_RGB_SMD_6028_2.8x3.5mm_Square" (at 99.06 177.8 0)
       (effects (font (size 1.27 1.27)) hide)
     )
@@
       (effects (font (size 1.27 1.27)) (justify left))
     )
-    (property "Footprint" "acheron_Components:LED_RGB_SMD_6028_2.8x3.5mm" (at 133.35 144.78 0)
+    (property "Footprint" "acheron_Components:LED_RGB_SMD_6028_2.8x3.5mm_Square" (at 133.35 144.78 0)
       (effects (font (size 1.27 1.27)) hide)
     )
@@
       (effects (font (size 1.27 1.27)) (justify left))
     )
-    (property "Footprint" "acheron_Components:LED_RGB_SMD_6028_2.8x3.5mm" (at 57.15 177.8 0)
+    (property "Footprint" "acheron_Components:LED_RGB_SMD_6028_2.8x3.5mm_Square" (at 57.15 177.8 0)
       (effects (font (size 1.27 1.27)) hide)
     )
@@
       (effects (font (size 1.27 1.27)) (justify left))
     )
-    (property "Footprint" "acheron_Components:LED_RGB_SMD_6028_2.8x3.5mm" (at 118.11 177.8 0)
+    (property "Footprint" "acheron_Components:LED_RGB_SMD_6028_2.8x3.5mm_Square" (at 118.11 177.8 0)
       (effects (font (size 1.27 1.27)) hide)
     )
@@
       (effects (font (size 1.27 1.27)) (justify left))
     )
-    (property "Footprint" "acheron_Components:LED_RGB_SMD_6028_2.8x3.5mm" (at 38.1 111.76 0)
+    (property "Footprint" "acheron_Components:LED_RGB_SMD_6028_2.8x3.5mm_Square" (at 38.1 111.76 0)
       (effects (font (size 1.27 1.27)) hide)
     )
@@
       (effects (font (size 1.27 1.27)) (justify left))
     )
-    (property "Footprint" "acheron_Components:LED_RGB_SMD_6028_2.8x3.5mm" (at 114.3 111.76 0)
+    (property "Footprint" "acheron_Components:LED_RGB_SMD_6028_2.8x3.5mm_Square" (at 114.3 111.76 0)
       (effects (font (size 1.27 1.27)) hide)
     )
@@
       (effects (font (size 1.27 1.27)) (justify left))
     )
-    (property "Footprint" "acheron_Components:LED_RGB_SMD_6028_2.8x3.5mm" (at 99.06 78.74 0)
+    (property "Footprint" "acheron_Components:LED_RGB_SMD_6028_2.8x3.5mm_Square" (at 99.06 78.74 0)
       (effects (font (size 1.27 1.27)) hide)
     )
@@
       (effects (font (size 1.27 1.27)) (justify left))
     )
-    (property "Footprint" "acheron_Components:LED_RGB_SMD_6028_2.8x3.5mm" (at 114.3 45.72 0)
+    (property "Footprint" "acheron_Components:LED_RGB_SMD_6028_2.8x3.5mm_Square" (at 114.3 45.72 0)
       (effects (font (size 1.27 1.27)) hide)
     )
@@
       (effects (font (size 1.27 1.27)) (justify left))
     )
-    (property "Footprint" "acheron_Components:LED_RGB_SMD_6028_2.8x3.5mm" (at 133.35 45.72 0)
+    (property "Footprint" "acheron_Components:LED_RGB_SMD_6028_2.8x3.5mm_Square" (at 133.35 45.72 0)
       (effects (font (size 1.27 1.27)) hide)
     )
@@
       (effects (font (size 1.27 1.27)) (justify left))
     )
-    (property "Footprint" "acheron_Components:LED_RGB_SMD_6028_2.8x3.5mm" (at 76.2 111.76 0)
+    (property "Footprint" "acheron_Components:LED_RGB_SMD_6028_2.8x3.5mm_Square" (at 76.2 111.76 0)
       (effects (font (size 1.27 1.27)) hide)
     )
@@
       (effects (font (size 1.27 1.27)) (justify left))
     )
-    (property "Footprint" "acheron_Components:LED_RGB_SMD_6028_2.8x3.5mm" (at 95.25 144.78 0)
+    (property "Footprint" "acheron_Components:LED_RGB_SMD_6028_2.8x3.5mm_Square" (at 95.25 144.78 0)
       (effects (font (size 1.27 1.27)) hide)
     )
@@
       (effects (font (size 1.27 1.27)) (justify left))
     )
-    (property "Footprint" "acheron_Components:LED_RGB_SMD_6028_2.8x3.5mm" (at 95.25 45.72 0)
+    (property "Footprint" "acheron_Components:LED_RGB_SMD_6028_2.8x3.5mm_Square" (at 95.25 45.72 0)
       (effects (font (size 1.27 1.27)) hide)
     )
@@
       (effects (font (size 1.27 1.27)) (justify left))
     )
-    (property "Footprint" "acheron_Components:LED_RGB_SMD_6028_2.8x3.5mm" (at 76.2 144.78 0)
+    (property "Footprint" "acheron_Components:LED_RGB_SMD_6028_2.8x3.5mm_Square" (at 76.2 144.78 0)
       (effects (font (size 1.27 1.27)) hide)
     )
@@
       (effects (font (size 1.27 1.27)) (justify left))
     )
-    (property "Footprint" "acheron_Components:LED_RGB_SMD_6028_2.8x3.5mm" (at 38.1 177.8 0)
+    (property "Footprint" "acheron_Components:LED_RGB_SMD_6028_2.8x3.5mm_Square" (at 38.1 177.8 0)
       (effects (font (size 1.27 1.27)) hide)
     )
@@
       (effects (font (size 1.27 1.27)) (justify left))
     )
-    (property "Footprint" "acheron_Components:LED_RGB_SMD_6028_2.8x3.5mm" (at 76.2 45.72 0)
+    (property "Footprint" "acheron_Components:LED_RGB_SMD_6028_2.8x3.5mm_Square" (at 76.2 45.72 0)
       (effects (font (size 1.27 1.27)) hide)
     )
@@
       (effects (font (size 1.27 1.27)) (justify left))
     )
-    (property "Footprint" "acheron_Components:LED_RGB_SMD_6028_2.8x3.5mm" (at 158.75 45.72 0)
+    (property "Footprint" "acheron_Components:LED_RGB_SMD_6028_2.8x3.5mm_Square" (at 158.75 45.72 0)
       (effects (font (size 1.27 1.27)) hide)
     )
@@
       (effects (font (size 1.27 1.27)) (justify left))
     )
-    (property "Footprint" "acheron_Components:LED_RGB_SMD_6028_2.8x3.5mm" (at 118.11 78.74 0)
+    (property "Footprint" "acheron_Components:LED_RGB_SMD_6028_2.8x3.5mm_Square" (at 118.11 78.74 0)
       (effects (font (size 1.27 1.27)) hide)
     )
@@
       (effects (font (size 1.27 1.27)) (justify left))
     )
-    (property "Footprint" "acheron_Components:LED_RGB_SMD_6028_2.8x3.5mm" (at 57.15 144.78 0)
+    (property "Footprint" "acheron_Components:LED_RGB_SMD_6028_2.8x3.5mm_Square" (at 57.15 144.78 0)
       (effects (font (size 1.27 1.27)) hide)
     )
@@
       (effects (font (size 1.27 1.27)) (justify left))
     )
-    (property "Footprint" "acheron_Components:LED_RGB_SMD_6028_2.8x3.5mm" (at 114.3 144.78 0)
+    (property "Footprint" "acheron_Components:LED_RGB_SMD_6028_2.8x3.5mm_Square" (at 114.3 144.78 0)
       (effects (font (size 1.27 1.27)) hide)
     )
@@
       (effects (font (size 1.27 1.27)) (justify left))
     )
-    (property "Footprint" "acheron_Components:LED_RGB_SMD_6028_2.8x3.5mm" (at 38.1 78.74 0)
+    (property "Footprint" "acheron_Components:LED_RGB_SMD_6028_2.8x3.5mm_Square" (at 38.1 78.74 0)
       (effects (font (size 1.27 1.27)) hide)
     )
@@
       (effects (font (size 1.27 1.27)) (justify left))
     )
-    (property "Footprint" "acheron_Components:LED_RGB_SMD_6028_2.8x3.5mm" (at 76.2 177.8 0)
-      (effects (font (size 1.27 1.27)) hide)
-    )
+    (property "Footprint" "acheron_Components:LED_RGB_SMD_6028_2.8x3.5mm_Square" (at 76.2 177.8 0)
+      (effects (font (size 1.27 1.27)) hide)
+    )
