File: kicad/kingslayer-28/rgb.kicad_sch (KiCad schematic)
At the start: 36 parts, among them IC2 IS31FL3731-QFLS2-TR

Commit message: fix RGB
Parts:
- D29, D30, D31, D32, D33, D34, D35, D36, D37, D38, D39, D40, D41, D42, D43, D44, D45, D46, D47, D48, D49, D50, D51, D52, D53, D54, D55, D56: symbol Device:LED_RGBA -> Device:LED_BAGR
Connections:
- net +5V: now also IC2.3 (SDB), R6.1
- net ca1: now also D29.4 (RK), D30.4 (RK), D31.4 (RK), D32.4 (RK), D33.4 (RK), D34.4 (RK), D36.2 (A), D41.2 (A); no longer D29.1 (RK), D30.1 (RK), D31.1 (RK), D32.1 (RK), D33.1 (RK), D34.1 (RK), D36.4 (A), D41.4 (A)
- net ca2: now also D29.3 (GK), D30.3 (GK), D31.3 (GK), D32.3 (GK), D33.3 (GK), D34.3 (GK), D37.2 (A), D42.2 (A); no longer D29.2 (GK), D30.2 (GK), D31.2 (GK), D32.2 (GK), D33.2 (GK), D34.2 (GK), D37.4 (A), D42.4 (A)
- net ca3: now also D29.1 (BK), D30.1 (BK), D31.1 (BK), D32.1 (BK), D33.1 (BK), D34.1 (BK), D38.2 (A), D43.2 (A); no longer D29.3 (BK), D30.3 (BK), D31.3 (BK), D32.3 (BK), D33.3 (BK), D34.3 (BK), D38.4 (A), D43.4 (A)
- net ca4: now also D29.2 (A), D36.4 (RK), D37.4 (RK), D38.4 (RK), D39.4 (RK), D40.4 (RK), D44.2 (A); no longer D29.4 (A), D36.1 (RK), D37.1 (RK), D38.1 (RK), D39.1 (RK), D40.1 (RK), D44.4 (A)
- net ca5: now also D30.2 (A), D36.3 (GK), D37.3 (GK), D38.3 (GK), D39.3 (GK), D40.3 (GK), D45.2 (A); no longer D30.4 (A), D36.2 (GK), D37.2 (GK), D38.2 (GK), D39.2 (GK), D40.2 (GK), D45.4 (A)
- net ca6: now also D31.2 (A), D36.1 (BK), D37.1 (BK), D38.1 (BK), D39.1 (BK), D40.1 (BK); no longer D31.4 (A), D36.3 (BK), D37.3 (BK), D38.3 (BK), D39.3 (BK), D40.3 (BK)
- net ca7: now also D32.2 (A), D39.2 (A), D41.4 (RK), D42.4 (RK), D43.4 (RK), D44.4 (RK), D45.4 (RK); no longer D32.4 (A), D39.4 (A), D41.1 (RK), D42.1 (RK), D43.1 (RK), D44.1 (RK), D45.1 (RK)
- net ca8: now also D33.2 (A), D40.2 (A), D41.3 (GK), D42.3 (GK), D43.3 (GK), D44.3 (GK), D45.3 (GK); no longer D33.4 (A), D40.4 (A), D41.2 (GK), D42.2 (GK), D43.2 (GK), D44.2 (GK), D45.2 (GK)
- net ca9: now also D34.2 (A), D41.1 (BK), D42.1 (BK), D43.1 (BK), D44.1 (BK), D45.1 (BK); no longer D34.4 (A), D41.3 (BK), D42.3 (BK), D43.3 (BK), D44.3 (BK), D45.3 (BK)
- net cb1: now also D35.2 (A), D46.4 (RK), D47.4 (RK), D48.4 (RK), D49.4 (RK), D50.4 (RK), D51.4 (RK), D52.2 (A); no longer D35.4 (A), D46.1 (RK), D47.1 (RK), D48.1 (RK), D49.1 (RK), D50.1 (RK), D51.1 (RK), D52.4 (A)
- net cb2: now also D46.3 (GK), D47.3 (GK), D48.3 (GK), D49.3 (GK), D50.3 (GK), D51.3 (GK), D53.2 (A); no longer D46.2 (GK), D47.2 (GK), D48.2 (GK), D49.2 (GK), D50.2 (GK), D51.2 (GK), D53.4 (A)
- net cb3: now also D46.1 (BK), D47.1 (BK), D48.1 (BK), D49.1 (BK), D50.1 (BK), D51.1 (BK), D54.2 (A); no longer D46.3 (BK), D47.3 (BK), D48.3 (BK), D49.3 (BK), D50.3 (BK), D51.3 (BK), D54.4 (A)
- net cb4: now also D46.2 (A), D52.4 (RK), D53.4 (RK), D54.4 (RK), D55.4 (RK), D56.4 (RK); no longer D46.4 (A), D52.1 (RK), D53.1 (RK), D54.1 (RK), D55.1 (RK), D56.1 (RK)
- net cb5: now also D47.2 (A), D52.3 (GK), D53.3 (GK), D54.3 (GK), D55.3 (GK), D56.3 (GK); no longer D47.4 (A), D52.2 (GK), D53.2 (GK), D54.2 (GK), D55.2 (GK), D56.2 (GK)
- net cb6: now also D48.2 (A), D52.1 (BK), D53.1 (BK), D54.1 (BK), D55.1 (BK), D56.1 (BK); no longer D48.4 (A), D52.3 (BK), D53.3 (BK), D54.3 (BK), D55.3 (BK), D56.3 (BK)
- net cb7: now also D35.4 (RK), D49.2 (A), D55.2 (A); no longer D35.1 (RK), D49.4 (A), D55.4 (A)
- net cb8: now also D35.3 (GK), D50.2 (A), D56.2 (A); no longer D35.2 (GK), D50.4 (A), D56.4 (A)
- net cb9: now also D35.1 (BK), D51.2 (A); no longer D35.3 (BK), D51.4 (A)
- net sdb: no longer IC2.3 (SDB), R6.1
Other:
- moved on the sheet: R6

Commit message: ERC
Changed lines of the file:
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@@
-    (stroke (width 0) (type default))
-  )
-  (wire (pts (xy 191.77 139.7) (xy 212.09 139.7))
     (stroke (width 0) (type default))
   )
@@
     )
   )
-  (global_label "sdb" (shape input) (at 212.09 139.7 0) (fields_autoplaced)
-    (effects (font (size 1.27 1.27)) (justify left))
-    (property "Intersheetrefs" "${INTERSHEET_REFS}" (at 218.4013 139.7 0)
-      (effects (font (size 1.27 1.27)) (justify left) hide)
-    )
-  )
